Commit message: feat(description): add the G-shape base under the arm
The arm floated 140 mm over the Gazebo ground: base_link (the bottom of the Jetson
casing) was lifted by BASE_HEIGHT_MM with nothing underneath.

- new g_base link: world -> g_base -> base_link, base_link on top of the plate
  (g_base_height = 0.032 m, from the vendor mesh; to measure)
- meshes/arm/g_base.dae from Elephant Robotics mycobot_280_pi/G_base.dae (BSD-2-Clause),
  turned 90 deg to line up with the casing; collision is a box of the same size
- tests: g_base frame required, zero-pose tool0 height updated

File: ros2_ws/src/braco_description/urdf/braco.urdf.xacro (robot description, xacro)
@@ -3,8 +3,8 @@
   braco: the whole robot. myCobot 280 + adaptive gripper + camera mount, with the TF frames
   the rest of the system uses (REP-103/105):
-    world -> base_link -> link1 ... link6 -> tool0 -> gripper_base ...
-                                              tool0 -> tcp
-                                              tool0 -> camera_mount -> camera_link
-                                                                        -> camera_optical_frame
+    world -> g_base -> base_link -> link1 ... link6 -> tool0 -> gripper_base ...
+                                                        tool0 -> tcp
+                                                        tool0 -> camera_mount -> camera_link
+                                                                                  -> camera_optical_frame
   Offsets marked MEASURE are not measured yet: they are zero or a rough value until someone
   puts calipers on the real hardware (docs/urdf-sim-to-real.md, "Open items").
@@ -25,8 +25,12 @@
       controllers="$(find braco_description)/config/gazebo_controllers.yaml"/>
   </xacro:if>
-  <!-- world: the table surface under the arm. Height of the arm's base over it, in metres.
-       Value from BASE_HEIGHT_MM of libs/cpp/includes/mycobot.hpp (table -> arm base, with the
-       Jetson casing / G-base). MEASURE again if the arm sits on something else. -->
-  <xacro:property name="base_height" value="0.140"/>
+  <!-- world: the table surface. The arm stands on the G-shape base (a 150 x 110 mm plate,
+       clamped to the table with its black grip), and base_link (the bottom of the Jetson casing)
+       sits on top of the plate. Plate thickness from the vendor mesh (meshes/arm/g_base.dae,
+       Elephant Robotics mycobot_280_pi/G_base.dae). MEASURE with calipers. -->
+  <xacro:property name="g_base_height" value="0.032"/>
+  <!-- UNMEASURED: weigh the plate. It is fixed to the world, so only the positive-mass rule
+       of the model (Gazebo, MoveIt) needs it. -->
+  <xacro:property name="g_base_mass" value="0.5"/>
   <!-- tcp: the point between the fingertips, along the tool0 z axis. Rough: the flange-to-tip
        length of the closed gripper with camera (TOOL_LENGTH_MM in mycobot.hpp). MEASURE to the
@@ -38,6 +42,35 @@
   <xacro:property name="camera_rpy" value="0 0 0"/>
   <link name="world"/>
-  <xacro:mycobot_280 parent="world">
-    <origin xyz="0 0 ${base_height}" rpy="0 0 0"/>
+  <!-- G-base: its frame is on the table, under the arm's axis. The vendor mesh is turned 90 deg
+       so its long side runs along y, like the Jetson casing. Collision is a box of the same size
+       (the mesh has 40k vertices and the plate never moves). -->
+  <link name="g_base">
+    <visual>
+      <origin xyz="0 0 0" rpy="0 0 ${pi / 2}"/>
+      <geometry>
+        <mesh filename="package://braco_description/meshes/arm/g_base.dae"/>
+      </geometry>
+    </visual>
+    <collision>
+      <origin xyz="0 0 ${g_base_height / 2}" rpy="0 0 0"/>
+      <geometry>
+        <box size="0.110 0.150 ${g_base_height}"/>
+      </geometry>
+    </collision>
+    <inertial>
+      <origin xyz="0 0 ${g_base_height / 2}" rpy="0 0 0"/>
+      <mass value="${g_base_mass}"/>
+      <inertia ixx="${g_base_mass * (0.150 ** 2 + g_base_height ** 2) / 12}" ixy="0" ixz="0"
+               iyy="${g_base_mass * (0.110 ** 2 + g_base_height ** 2) / 12}" iyz="0"
+               izz="${g_base_mass * (0.110 ** 2 + 0.150 ** 2) / 12}"/>
+    </inertial>
+  </link>
+  <joint name="world_to_g_base" type="fixed">
+    <parent link="world"/>
+    <child link="g_base"/>
+    <origin xyz="0 0 0" rpy="0 0 0"/>
+  </joint>
+  <xacro:mycobot_280 parent="g_base">
+    <origin xyz="0 0 ${g_base_height}" rpy="0 0 0"/>
   </xacro:mycobot_280>
   <!-- tool0: the flange, z pointing out of it (REP-103 / ROS-Industrial name). Same frame as link6. -->

Commit message: fix(mycobot): use Jetson Nano kinematics in the table-clearance check
minHeightMm() used the joint origins of the myCobot 280 M5 (J1 0.13156 m above a short
base) with BASE_HEIGHT_MM, the height of the top of the Jetson casing. Every height it
computed was about 85 mm too high: with the arm straight out (J2 -90) it saw the tool
96 mm above the table instead of 11 mm, and allowed the move.

- J1/J2 origins of the Jetson Nano arm (0.15756, -0.001), the same as braco_description
- the chain starts at the bottom of the casing: BASE_HEIGHT_MM (140, measured: table to
  the top of the casing, G-base included) - CASING_HEIGHT_MM (109.7, vendor mesh)
- URDF: g_base_height 0.030 to match (vendor mount height, 30.3 mm measured)
- test_urdf.py: the C++ joint origins and base height must match the URDF

File: ros2_ws/src/braco_description/urdf/braco.urdf.xacro (robot description, xacro)
@@ -27,7 +27,12 @@
   <!-- world: the table surface. The arm stands on the G-shape base (a 150 x 110 mm plate,
        clamped to the table with its black grip), and base_link (the bottom of the Jetson casing)
-       sits on top of the plate. Plate thickness from the vendor mesh (meshes/arm/g_base.dae,
-       Elephant Robotics mycobot_280_pi/G_base.dae). MEASURE with calipers. -->
-  <xacro:property name="g_base_height" value="0.032"/>
+       sits on top of the plate, 2 mm down in its pocket. Measured: table -> top of the casing
+       = 140 mm (BASE_HEIGHT_MM in libs/cpp/includes/mycobot.hpp), minus the 109.7 mm casing
+       (CASING_HEIGHT_MM) = 30.3 mm; the vendor mounts it at 30 mm (mycobot_280_pi URDF).
+       test_urdf.py keeps g_base_height and mycobot.hpp within 1 mm. -->
+  <xacro:property name="g_base_height" value="0.030"/>
+  <!-- Plate thickness, from the vendor mesh (meshes/arm/g_base.dae, Elephant Robotics
+       mycobot_280_pi/G_base.dae). Only for the collision box and the inertia. -->
+  <xacro:property name="g_base_thickness" value="0.032"/>
   <!-- UNMEASURED: weigh the plate. It is fixed to the world, so only the positive-mass rule
        of the model (Gazebo, MoveIt) needs it. -->
@@ -53,14 +58,14 @@
     </visual>
     <collision>
-      <origin xyz="0 0 ${g_base_height / 2}" rpy="0 0 0"/>
+      <origin xyz="0 0 ${g_base_thickness / 2}" rpy="0 0 0"/>
       <geometry>
-        <box size="0.110 0.150 ${g_base_height}"/>
+        <box size="0.110 0.150 ${g_base_thickness}"/>
       </geometry>
     </collision>
     <inertial>
-      <origin xyz="0 0 ${g_base_height / 2}" rpy="0 0 0"/>
+      <origin xyz="0 0 ${g_base_thickness / 2}" rpy="0 0 0"/>
       <mass value="${g_base_mass}"/>
-      <inertia ixx="${g_base_mass * (0.150 ** 2 + g_base_height ** 2) / 12}" ixy="0" ixz="0"
-               iyy="${g_base_mass * (0.110 ** 2 + g_base_height ** 2) / 12}" iyz="0"
+      <inertia ixx="${g_base_mass * (0.150 ** 2 + g_base_thickness ** 2) / 12}" ixy="0" ixz="0"
+               iyy="${g_base_mass * (0.110 ** 2 + g_base_thickness ** 2) / 12}" iyz="0"
                izz="${g_base_mass * (0.110 ** 2 + 0.150 ** 2) / 12}"/>
     </inertial>

Commit message: fix(description): turn the flange and gripper 45 degrees to match the real arm
At joint 6 = 0 the flange's LEGO hole grid on the real arm is turned 45 degrees from the
vendor model, so the gripper pinned to it looked twisted in Gazebo. New flange_yaw
(-45, checked against the real arm) turns the flange mesh and tool0 about the joint 6
axis; the gripper, tcp and camera frames follow, so the pins stay in the flange holes.
Positions do not change.

File: ros2_ws/src/braco_description/urdf/braco.urdf.xacro (robot description, xacro)
@@ -46,4 +46,10 @@
   <xacro:property name="camera_xyz" value="0 0 0"/>
   <xacro:property name="camera_rpy" value="0 0 0"/>
+  <!-- Flange angle about the joint 6 axis, degrees. The flange's LEGO hole grid on the real arm
+       is turned 45 deg from the vendor model at joint 6 = 0 (compared side by side with the real
+       arm). Turns the flange mesh and tool0, and with tool0 everything on it (gripper, tcp,
+       camera), so the gripper's pins stay in the flange holes. Positions do not change.
+       Checked in Gazebo against the real arm: -45. -->
+  <xacro:property name="flange_yaw" value="-45"/>
   <link name="world"/>
   <!-- G-base: its frame is on the table, under the arm's axis. The vendor mesh is turned 90 deg
@@ -76,13 +82,14 @@
     <origin xyz="0 0 0" rpy="0 0 0"/>
   </joint>
-  <xacro:mycobot_280 parent="g_base">
+  <xacro:mycobot_280 parent="g_base" flange_yaw="${radians(flange_yaw)}">
     <origin xyz="0 0 ${g_base_height}" rpy="0 0 0"/>
   </xacro:mycobot_280>
-  <!-- tool0: the flange, z pointing out of it (REP-103 / ROS-Industrial name). Same frame as link6. -->
+  <!-- tool0: the flange, z pointing out of it (REP-103 / ROS-Industrial name). link6 turned by
+       flange_yaw about z, so x and y follow the flange holes. -->
   <link name="tool0"/>
   <joint name="link6_to_tool0" type="fixed">
     <parent link="link6"/>
     <child link="tool0"/>
-    <origin xyz="0 0 0" rpy="0 0 0"/>
+    <origin xyz="0 0 0" rpy="0 0 ${radians(flange_yaw)}"/>
   </joint>
   <xacro:adaptive_gripper parent="tool0" actuated="$(arg gripper_actuated)">

File: ros2_ws/src/braco_description/urdf/mycobot_280.urdf.xacro (robot description, xacro)
@@ -68,5 +68,6 @@
     </joint>
   </xacro:macro>
-  <xacro:macro name="mycobot_280" params="parent:=world *origin">
+  <!-- flange_yaw (rad): turns the flange mesh about the joint 6 axis (see braco.urdf.xacro). -->
+  <xacro:macro name="mycobot_280" params="parent:=world flange_yaw:=0 *origin">
     <xacro:arm_link name="base_link" mesh="base_link" mass="${base_mass}"
                     xyz="0 0 0" rpy="0 0 3.14159"/>
@@ -87,5 +88,5 @@
                     xyz="0 0 -0.038" rpy="0 0 0"/>
     <xacro:arm_link name="link6" mesh="link6" mass="${link_mass}"
-                    xyz="0 0 -0.012" rpy="0 0 0"/>
+                    xyz="0 0 -0.012" rpy="0 0 ${flange_yaw}"/>
     <xacro:arm_joint n="1" parent="base_link" child="link1"
                      xyz="0 0 0.15756" rpy="0 0 0"/>
