Commit message: feat(description): measured velocities, documented masses, payload-based efforts, camera flange
- joint velocity limits measured on the real arm at speed 100:
  2.64 / 2.44 / 2.72 / 2.69 / 2.65 / 2.60 rad/s (speed setting: 0.0265 rad/s per unit)
- masses from documented totals (no scale): gripper 110 g, arm 1.03 kg split by mesh
  volume; camera plate 40 g estimated
- effort limits: no published servo torque, so the lower bound the rated 0.25 kg payload
  implies in each joint's worst pose: 1.9 / 1.9 / 1.2 / 0.7 / 0.6 / 0.6 N*m
- camera: Elephant Robotics' camera flange (mesh and mount from the vendor's
  mycobot_280_pi model, BSD-2-Clause), between the flange and the gripper; camera_link
  on the lens at (41.5, 0, 12) mm in tool0, looking along tool0 z; the gripper moves out
  by the plate's 16.3 mm

File: ros2_ws/src/braco_description/urdf/adaptive_gripper.xacro (robot description, xacro)
@@ -12,7 +12,10 @@
 -->
 <robot xmlns:xacro="http://www.ros.org/wiki/xacro">
-  <!-- UNMEASURED placeholders (weigh the gripper on a scale, see docs/urdf-sim-to-real.md) -->
-  <xacro:property name="gripper_base_mass" value="0.1"/>
-  <xacro:property name="finger_link_mass" value="0.01"/>
+  <!-- Total 110 g: the myCobot Adaptive Gripper's documented weight (retailer spec sheets; the
+       same listings give the 110 x 90 x 60 mm and 150 g clamp printed on our gripper's label).
+       The split is ESTIMATED: body 80 g (it holds the servo), each of the 6 finger parts 5 g.
+       Replace with a scale reading when one is available. -->
+  <xacro:property name="gripper_base_mass" value="0.080"/>
+  <xacro:property name="finger_link_mass" value="0.005"/>
   <xacro:macro name="finger_link" params="name mass xyz">
     <link name="${name}">

File: ros2_ws/src/braco_description/urdf/braco.urdf.xacro (robot description, xacro)
@@ -42,8 +42,20 @@
        middle of the closed fingertips. -->
   <xacro:property name="tcp_length" value="0.130"/>
-  <!-- camera mount on the flange. MEASURE with calipers: position of the camera lens centre in
-       the tool0 frame (x, y, z in metres). camera_link follows REP-103: x forward, y left, z up. -->
-  <xacro:property name="camera_xyz" value="0 0 0"/>
-  <xacro:property name="camera_rpy" value="0 0 0"/>
+  <!-- Camera: Elephant Robotics' camera flange (in the arm's box, docs/inventory), a 83 x 34 mm
+       plate, 16 mm thick with the camera module. Its LEGO hole grid goes on the flange's and the
+       gripper pins onto the same holes on its front face: flange -> camera plate -> gripper. The
+       lens is at the other end of the plate, on the gripper side. Mesh and mount from the vendor
+       (mycobot_280_pi/camera_flange.dae, mycobot_280_pi_with_camera_flange.urdf); the plate's
+       direction (tool0 +x) matches the real arm's photos at the zero pose. -->
+  <xacro:property name="camera_plate_thickness" value="0.0163"/>
+  <!-- ESTIMATED (no scale): the plate and the USB camera module. -->
+  <xacro:property name="camera_mass" value="0.040"/>
+  <!-- camera_link at the lens, in camera_mount (= tool0 axes), from the vendor mesh: lens centre
+       41.5 mm out along the plate, the lens glass 12 mm from the flange face. It looks along
+       tool0 +z, like the gripper; camera_link follows REP-103 (x forward), so x = tool0 z.
+       The roll of the image (camera_link about its x) is not known from the model: the hand-eye
+       calibration sets it. -->
+  <xacro:property name="camera_xyz" value="0.0415 0 0.012"/>
+  <xacro:property name="camera_rpy" value="0 ${-pi / 2} 0"/>
   <!-- Flange angle about the joint 6 axis, degrees. The flange's LEGO hole grid on the real arm
        is turned 45 deg from the vendor model at joint 6 = 0 (compared side by side with the real
@@ -93,6 +105,8 @@
     <origin xyz="0 0 0" rpy="0 0 ${radians(flange_yaw)}"/>
   </joint>
+  <!-- The gripper on the camera plate's front face: the vendor's flange mount (0.034) moved out by
+       the plate's thickness. -->
   <xacro:adaptive_gripper parent="tool0" actuated="$(arg gripper_actuated)">
-    <origin xyz="0 0 0.034" rpy="${pi / 2} 0 0"/>
+    <origin xyz="0 0 ${0.034 + camera_plate_thickness}" rpy="${pi / 2} 0 0"/>
   </xacro:adaptive_gripper>
   <link name="tcp"/>
@@ -102,9 +116,31 @@
     <origin xyz="0 0 ${tcp_length}" rpy="0 0 0"/>
   </joint>
-  <link name="camera_mount"/>
+  <!-- camera_mount: the camera plate, frame on tool0's axes. The visual origin is the vendor's
+       joint (0 0 0.01, rpy pi/2 0 0) times its mesh offset (0.024 -0.008 0, rpy 0 pi 0). -->
+  <link name="camera_mount">
+    <visual>
+      <origin xyz="0.024 0 0.002" rpy="${pi / 2} 0 ${pi}"/>
+      <geometry>
+        <mesh filename="package://braco_description/meshes/arm/camera_flange.dae"/>
+      </geometry>
+    </visual>
+    <collision>
+      <origin xyz="0.024 0.0005 0.010" rpy="0 0 0"/>
+      <geometry>
+        <box size="0.083 0.034 0.016"/>
+      </geometry>
+    </collision>
+    <inertial>
+      <origin xyz="0.024 0 0.010" rpy="0 0 0"/>
+      <mass value="${camera_mass}"/>
+      <inertia ixx="${camera_mass * (0.034 ** 2 + 0.016 ** 2) / 12}" ixy="0" ixz="0"
+               iyy="${camera_mass * (0.083 ** 2 + 0.016 ** 2) / 12}" iyz="0"
+               izz="${camera_mass * (0.083 ** 2 + 0.034 ** 2) / 12}"/>
+    </inertial>
+  </link>
   <joint name="tool0_to_camera_mount" type="fixed">
     <parent link="tool0"/>
     <child link="camera_mount"/>
-    <origin xyz="${camera_xyz}" rpy="${camera_rpy}"/>
+    <origin xyz="0 0 0" rpy="0 0 0"/>
   </joint>
   <link name="camera_link"/>
@@ -112,5 +148,5 @@
     <parent link="camera_mount"/>
     <child link="camera_link"/>
-    <origin xyz="0 0 0" rpy="0 0 0"/>
+    <origin xyz="${camera_xyz}" rpy="${camera_rpy}"/>
   </joint>
   <!-- Optical frame: z forward, x right, y down (REP-103). Rotated from camera_link. -->

File: ros2_ws/src/braco_description/urdf/mycobot_280.urdf.xacro (robot description, xacro)
@@ -21,11 +21,21 @@
   <xacro:property name="limit_min" value="${[-166.0, -138.0, -149.0, -149.0, -153.0, -178.0]}"/>
   <xacro:property name="limit_max" value="${[166.0, 138.0, 149.0, 149.0, 158.0, 178.0]}"/>
-  <!-- UNMEASURED placeholders: see docs/urdf-sim-to-real.md, "Open items".
-       velocity rad/s (to measure per joint), effort N*m (servo stall torque, datasheet),
-       masses kg (to weigh / vendor data). Nothing in the system depends on them yet. -->
-  <xacro:property name="joint_velocity" value="1.0"/>
-  <xacro:property name="joint_effort" value="1.0"/>
-  <xacro:property name="base_mass" value="0.4"/>
-  <xacro:property name="link_mass" value="0.1"/>
+  <!-- Joint velocity limits, rad/s, J1..J6: MEASURED on the real arm at speed 100
+       (sim_to_real.py velocity, middle 80 % of a -A..+A sweep; docs/urdf-sim-to-real.md).
+       joint3 measured 2.79 average but 2.72 peak (a 0.6 s sweep at 20 Hz joint states):
+       the lower one is used. The firmware speed setting scales linearly: rad/s = 0.0265 x speed. -->
+  <xacro:property name="joint_velocity" value="${[2.64, 2.44, 2.72, 2.69, 2.65, 2.60]}"/>
+  <!-- Effort limits, N*m, J1..J6: APPROXIMATION. Elephant Robotics does not publish the joint
+       servos' torque, so this is the lower bound the published spec implies: the static torque
+       to hold the arm (masses below) plus the rated 0.25 kg payload at tcp in each joint's worst
+       pose (J2 1.89, J3 1.15, J4 0.67, J5 0.57, with the camera plate), rounded up. J1 and J6 carry no gravity load and
+       take their neighbour's value. Replace with stall torques if a datasheet turns up. -->
+  <xacro:property name="joint_effort" value="${[1.9, 1.9, 1.2, 0.7, 0.6, 0.6]}"/>
+  <!-- Masses, kg. ESTIMATED from documented totals (no scale yet, see docs/urdf-sim-to-real.md):
+       whole arm 1.03 kg (myCobot 280 Jetson Nano spec sheet); moving links 1..6 about 0.65 kg
+       (the standard 280 is 850 g with a ~0.2 kg M5 base), split by mesh volume
+       (21 / 35 / 27 / 3 / 12 / 2 %); base_link (Jetson casing) the rest. -->
+  <xacro:property name="base_mass" value="0.38"/>
+  <xacro:property name="link_masses" value="${[0.14, 0.23, 0.17, 0.02, 0.08, 0.01]}"/>
   <!-- Solid cylinder around the link z axis, centred on the link frame. UNMEASURED: radius and
        length are rough; the point is a positive-definite inertia (Gazebo and MoveIt need one). -->
@@ -65,5 +75,5 @@
       <axis xyz="0 0 1"/>
       <limit lower="${radians(limit_min[n - 1])}" upper="${radians(limit_max[n - 1])}"
-             velocity="${joint_velocity}" effort="${joint_effort}"/>
+             velocity="${joint_velocity[n - 1]}" effort="${joint_effort[n - 1]}"/>
     </joint>
   </xacro:macro>
@@ -77,15 +87,15 @@
       <xacro:insert_block name="origin"/>
     </joint>
-    <xacro:arm_link name="link1" mesh="link1" mass="${link_mass}"
+    <xacro:arm_link name="link1" mesh="link1" mass="${link_masses[0]}"
                     xyz="0 0 -0.06096" rpy="0 0 -1.5708"/>
-    <xacro:arm_link name="link2" mesh="link2" mass="${link_mass}"
+    <xacro:arm_link name="link2" mesh="link2" mass="${link_masses[1]}"
                     xyz="0 0 0.03256" rpy="0 -1.5708 0"/>
-    <xacro:arm_link name="link3" mesh="link3" mass="${link_mass}"
+    <xacro:arm_link name="link3" mesh="link3" mass="${link_masses[2]}"
                     xyz="0 0 0.03056" rpy="0 -1.5708 0"/>
-    <xacro:arm_link name="link4" mesh="link4" mass="${link_mass}"
+    <xacro:arm_link name="link4" mesh="link4" mass="${link_masses[3]}"
                     xyz="0 0 -0.03356" rpy="0 -1.5708 1.5708"/>
-    <xacro:arm_link name="link5" mesh="link5" mass="${link_mass}"
+    <xacro:arm_link name="link5" mesh="link5" mass="${link_masses[4]}"
                     xyz="0 0 -0.038" rpy="0 0 0"/>
-    <xacro:arm_link name="link6" mesh="link6" mass="${link_mass}"
+    <xacro:arm_link name="link6" mesh="link6" mass="${link_masses[5]}"
                     xyz="0 0 -0.012" rpy="0 0 ${flange_yaw}"/>
     <xacro:arm_joint n="1" parent="base_link" child="link1"

Commit message: fix: fixed gripper 3D model for gazebo

File: ros2_ws/src/braco_description/urdf/adaptive_gripper.xacro (robot description, xacro)
@@ -17,4 +17,9 @@
        Replace with a scale reading when one is available. -->
   <xacro:property name="gripper_base_mass" value="0.080"/>
+  <!-- gripper_controller (the master) range, rad: closed (tips 3.6 mm apart) .. open. The five
+       followers get exactly this range times their mimic multiplier: the vendor's own follower
+       limits were narrower (e.g. -0.5..0.5), so they could not follow the master to its ends. -->
+  <xacro:property name="gripper_lower" value="-0.74"/>
+  <xacro:property name="gripper_upper" value="0.15"/>
   <xacro:property name="finger_link_mass" value="0.005"/>
   <xacro:macro name="finger_link" params="name mass xyz">
@@ -41,6 +46,7 @@
   </xacro:macro>
   <!-- One finger joint: fixed at 0 unless `actuated`; `mimic` = "" for the master joint,
-       "multiplier" for the others (they follow gripper_controller). -->
-  <xacro:macro name="finger_joint" params="name parent child xyz lower upper actuated mimic:=''">
+       "multiplier" for the others (they follow gripper_controller, limits from its range). -->
+  <xacro:macro name="finger_joint" params="name parent child xyz actuated mimic:=''">
+    <xacro:property name="m" value="${1.0 if mimic == '' else float(mimic)}"/>
     <xacro:if value="${actuated}">
       <joint name="${name}" type="revolute">
@@ -49,5 +55,6 @@
         <origin xyz="${xyz}" rpy="0 0 0"/>
         <axis xyz="0 0 1"/>
-        <limit lower="${lower}" upper="${upper}" velocity="1.0" effort="1.0"/>
+        <limit lower="${min(m * gripper_lower, m * gripper_upper)}"
+               upper="${max(m * gripper_lower, m * gripper_upper)}" velocity="1.0" effort="1.0"/>
         <xacro:if value="${mimic != ''}">
           <mimic joint="gripper_controller" multiplier="${mimic}" offset="0"/>
@@ -76,21 +83,25 @@
       <xacro:insert_block name="origin"/>
     </joint>
-    <!-- gripper_controller is the master; the other five follow it (vendor linkage) -->
+    <!-- gripper_controller is the master; the other five follow it (vendor linkage).
+         The four joints on gripper_base sit 7.5 mm lower than the vendor's (y 0.005 -> -0.0025,
+         0.027 -> 0.0195): each part's mesh offset is minus its pivot in the gripper frame, and the
+         body's front face has the central pins' holes at (+-5.5, 19.5) mm; the vendor values put
+         the whole linkage 7.5 mm above the body (checked against a photo of our gripper). -->
     <xacro:finger_joint name="gripper_controller" parent="gripper_base" child="gripper_left3"
-                        xyz="-0.012 0.005 0" lower="-0.74" upper="0.15" actuated="${actuated}"/>
+                        xyz="-0.012 -0.0025 0" actuated="${actuated}"/>
     <xacro:finger_joint name="gripper_base_to_gripper_left2" parent="gripper_base"
-                        child="gripper_left2" xyz="-0.005 0.027 0" lower="-0.8" upper="0.5"
+                        child="gripper_left2" xyz="-0.005 0.0195 0"
                         actuated="${actuated}" mimic="1.0"/>
     <xacro:finger_joint name="gripper_left3_to_gripper_left1" parent="gripper_left3"
-                        child="gripper_left1" xyz="-0.027 0.016 0" lower="-0.5" upper="0.5"
+                        child="gripper_left1" xyz="-0.027 0.016 0"
                         actuated="${actuated}" mimic="-1.0"/>
     <xacro:finger_joint name="gripper_base_to_gripper_right3" parent="gripper_base"
-                        child="gripper_right3" xyz="0.012 0.005 0" lower="-0.15" upper="0.7"
+                        child="gripper_right3" xyz="0.012 -0.0025 0"
                         actuated="${actuated}" mimic="-1.0"/>
     <xacro:finger_joint name="gripper_base_to_gripper_right2" parent="gripper_base"
-                        child="gripper_right2" xyz="0.005 0.027 0" lower="-0.5" upper="0.8"
+                        child="gripper_right2" xyz="0.005 0.0195 0"
                         actuated="${actuated}" mimic="-1.0"/>
     <xacro:finger_joint name="gripper_right3_to_gripper_right1" parent="gripper_right3"
-                        child="gripper_right1" xyz="0.027 0.016 0" lower="-0.5" upper="0.5"
+                        child="gripper_right1" xyz="0.027 0.016 0"
                         actuated="${actuated}" mimic="1.0"/>
   </xacro:macro>
